File: 5VTO3.3V.sch (KiCad schematic (older format))
At the start: 10 parts, among them IC1 TPS64202DBVT, IC2 SI2323DS-T1-E3

Commit message: Assigned PCB footprints to schematic symbols
Parts:
- 0.7, 120K1: footprint (none) -> Resistor_SMD:R_1206_3216Metric_Pad1.42x1.75mm_HandSolder
- 10u1, 47p1: footprint (none) -> Capacitor_SMD:C_1206_3216Metric_Pad1.42x1.75mm_HandSolder
- 210K: renamed from R1; footprint (none) -> Resistor_SMD:R_1206_3216Metric_Pad1.42x1.75mm_HandSolder
- 56u1: footprint (none) -> Inductor:LPS6235563MRC
- D1: footprint SOT95P285X140-6N -> Shottky:SOT95P285X140-6N
- IC1: footprint SOT95P280X145-6N -> Buck regulator:SOT95P280X145-6N
- IC2: footprint SOT95P237X112-3N -> P-MOSFET:SOT95P237X112-3N
- renumbered 470u1 to 470u
Changed lines of the file:
@@
 F 0 "IC1" H 3700 3250 50  0000 C CNN
 F 1 "TPS64202DBVT" H 3700 3150 50  0000 C CNN
-F 2 "SOT95P280X145-6N" H 4150 3050 50  0001 L CNN
+F 2 "Buck regulator:SOT95P280X145-6N" H 4150 3050 50  0001 L CNN
 F 3 "http://www.ti.com/lit/gpn/tps64202" H 4150 2950 50  0001 L CNN
 F 4 "Texas Instruments TPS64202DBVT, DC-DC Controller, 6.5 V Step-Down, 6-Pin, SOT-23" H 4150 2850 50  0001 L CNN "Description"
@@
 F 0 "D1" H 3650 5450 50  0000 C CNN
 F 1 "ZHCS2000TA" H 3650 5350 50  0000 C CNN
-F 2 "SOT95P285X140-6N" H 4000 5250 50  0001 L CNN
+F 2 "Shottky:SOT95P285X140-6N" H 4000 5250 50  0001 L CNN
 F 3 "https://componentsearchengine.com/Datasheets/1/ZHCS2000TA.pdf" H 4000 5150 50  0001 L CNN
 F 4 "Schottky diode 2A 40V SOT23, ZHCS2000TA Diodes Inc ZHCS2000TA, SMT Schottky Diode, 40V 2A, 5.5ns, 6-Pin SOT-23" H 4000 5050 50  0001 L CNN "Description"
@@
 F 0 "IC2" V 5300 3500 50  0000 L CNN
 F 1 "SI2323DS-T1-E3" V 5350 3500 50  0000 L CNN
-F 2 "SOT95P237X112-3N" H 5600 3450 50  0001 L CNN
+F 2 "P-MOSFET:SOT95P237X112-3N" H 5600 3450 50  0001 L CNN
 F 3 "https://datasheet.datasheetarchive.com/originals/distributors/Datasheets-DGA23/1580060.pdf" H 5600 3350 50  0001 L CNN
 F 4 "SI2323DS-T1-E3, P-channel MOSFET Transistor 3.7 A 20 V, 3-Pin SOT-23, TO-236" H 5600 3250 50  0001 L CNN "Description"
@@
 F 0 "0.7" H 4800 2200 50  0000 L CNN
 F 1 "R" H 4800 2150 50  0000 L CNN
-F 2 "" V 4630 2150 50  0001 C CNN
+F 2 "Resistor_SMD:R_1206_3216Metric_Pad1.42x1.75mm_HandSolder" V 4630 2150 50  0001 C CNN
 F 3 "~" H 4700 2150 50  0001 C CNN
 	1    4700 2150
@@
 F 0 "10u1" H 2200 2500 50  0000 L CNN
 F 1 "CAP" H 2200 2450 50  0000 L CNN
-F 2 "" H 2000 2450 50  0001 C CNN
+F 2 "Capacitor_SMD:C_1206_3216Metric_Pad1.42x1.75mm_HandSolder" H 2000 2450 50  0001 C CNN
 F 3 "" H 2000 2450 50  0001 C CNN
 	1    2000 2450
@@
 F 0 "56u1" H 5900 4750 50  0000 C CNN
 F 1 "INDUCTOR" H 5900 4650 50  0000 C CNN
-F 2 "" H 5900 4500 50  0001 C CNN
+F 2 "Inductor:LPS6235563MRC" H 5900 4500 50  0001 C CNN
 F 3 "" H 5900 4500 50  0001 C CNN
 	1    5900 4500
@@
 $EndComp
 $Comp
-L Device:R R1
+L Device:R 210K
 U 1 1 62A10215
 P 6850 5100
-F 0 "R1" H 6950 5150 50  0000 L CNN
+F 0 "210K" H 6950 5150 50  0000 L CNN
 F 1 "R" H 6950 5100 50  0000 L CNN
-F 2 "" V 6780 5100 50  0001 C CNN
+F 2 "Resistor_SMD:R_1206_3216Metric_Pad1.42x1.75mm_HandSolder" V 6780 5100 50  0001 C CNN
 F 3 "~" H 6850 5100 50  0001 C CNN
 	1    6850 5100
@@
 F 0 "120K1" H 6950 5850 50  0000 L CNN
 F 1 "R" H 6950 5800 50  0000 L CNN
-F 2 "" V 6780 5800 50  0001 C CNN
+F 2 "Resistor_SMD:R_1206_3216Metric_Pad1.42x1.75mm_HandSolder" V 6780 5800 50  0001 C CNN
 F 3 "~" H 6850 5800 50  0001 C CNN
 	1    6850 5800
@@
 F 0 "47p1" H 7900 5200 50  0000 L CNN
 F 1 "CAP" H 7900 5150 50  0000 L CNN
-F 2 "" H 7700 5150 50  0001 C CNN
+F 2 "Capacitor_SMD:C_1206_3216Metric_Pad1.42x1.75mm_HandSolder" H 7700 5150 50  0001 C CNN
 F 3 "" H 7700 5150 50  0001 C CNN
 	1    7700 5150
@@
 $EndComp
 $Comp
-L Device:CP1 470u1
+L Device:CP1 470u
 U 1 1 62A1048D
 P 8550 5450
-F 0 "470u1" H 8700 5500 50  0000 L CNN
+F 0 "470u" H 8700 5500 50  0000 L CNN
 F 1 "CP1" H 8700 5450 50  0000 L CNN
 F 2 "" H 8550 5450 50  0001 C CNN
